File: src/solder_challenge_555.kicad_pcb (KiCad board)
At the start: 4 copper layers, 43.2 x 25.5 mm, 25 parts, among them J1 USB_B_Micro, J2 Conn_01x04_Socket

Commit message: logo update
Other:
- board text removed: "Scan For BOM"

Commit message: v 1 dot 5 for real
i left the qr code off the back... woooo
Other:
- board text added: "Scan for BOM"
